File: eagle/keepuntil-v1.0/KeepUntil-v1.0.sch (EAGLE design)
At the start: 17 parts, among them IC2 REG1117, Q1 CSTCR6M00G53Z, T1 BC846, U1 ATMEGA328P-AU, X1 MINI-USB-32005-201

Commit message: pin header updates in schematic
Parts:
- added CONTROL: (no value), pinhead:PINHD-2X5
- added R3, R4, R5: 1K, resistor:R-EU_R0805
- added R6, R8, R9: 4.7K, resistor:R-EU_R0805
- KEYPAD: device pinhead:PINHD-2X3 -> adafruit:PINHD-2X4
Connections:
- removed net COL1: KEYPAD.2, U1.PB0
- removed net COL2: KEYPAD.4, U1.PB1
- removed net COL3: KEYPAD.6, U1.PB2
- removed net ROW1: KEYPAD.1, U1.PD5
- removed net ROW2: KEYPAD.3, U1.PD6
- removed net ROW3: KEYPAD.5, U1.PD7
- new net N$10: U1.PD7
- new net N$11: U1.PB0
- new net N$12: U1.PB1
- new net N$13: U1.PB2
- new net N$14: U1.PC3
- new net N$6: U1.PD5
- new net N$9: U1.PD6
- net LED-GRN: no longer U1.PC0
- net LED-RED: no longer U1.PC1
- net SERVO: no longer U1.ADC6
Changed lines of the file:
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@@
 <part name="R7" library="resistor" deviceset="R-EU_" device="R0805" value="330"/>
 <part name="ISP" library="pinhead" deviceset="PINHD-2X3" device=""/>
-<part name="KEYPAD" library="pinhead" deviceset="PINHD-2X3" device=""/>
 <part name="LOCK-CTRL" library="pinhead" deviceset="PINHD-2X4" device=""/>
 <part name="T1" library="transistor" deviceset="BC846" device=""/>
@@
 <part name="P+1" library="supply1" deviceset="VCC" device=""/>
 <part name="SERIAL" library="adafruit" deviceset="PINHD-1X3" device=""/>
-<part name="GND12" library="supply1" deviceset="GND" device=""/>
+<part name="GND3" library="supply1" deviceset="GND" device=""/>
+<part name="R3" library="resistor" deviceset="R-EU_" device="R0805" value="1K"/>
+<part name="R4" library="resistor" deviceset="R-EU_" device="R0805" value="1K"/>
+<part name="R5" library="resistor" deviceset="R-EU_" device="R0805" value="1K"/>
+<part name="R6" library="resistor" deviceset="R-EU_" device="R0805" value="4.7K"/>
+<part name="R8" library="resistor" deviceset="R-EU_" device="R0805" value="4.7K"/>
+<part name="R9" library="resistor" deviceset="R-EU_" device="R0805" value="4.7K"/>
+<part name="KEYPAD" library="adafruit" deviceset="PINHD-2X4" device=""/>
+<part name="CONTROL" library="pinhead" deviceset="PINHD-2X5" device=""/>
 </parts>
 <sheets>
@@
 <instance part="R7" gate="G$1" x="111.76" y="139.7" rot="R90"/>
 <instance part="ISP" gate="A" x="53.34" y="25.4"/>
-<instance part="KEYPAD" gate="A" x="53.34" y="78.74"/>
 <instance part="LOCK-CTRL" gate="A" x="53.34" y="50.8"/>
 <instance part="T1" gate="G$1" x="114.3" y="40.64"/>
@@
 <instance part="P+1" gate="VCC" x="121.92" y="147.32" rot="R270"/>
 <instance part="SERIAL" gate="A" x="53.34" y="104.14"/>
-<instance part="GND12" gate="1" x="43.18" y="93.98"/>
+<instance part="GND3" gate="1" x="43.18" y="93.98"/>
+<instance part="R3" gate="G$1" x="15.24" y="81.28" rot="R270"/>
+<instance part="R4" gate="G$1" x="25.4" y="81.28" rot="R270"/>
+<instance part="R5" gate="G$1" x="35.56" y="81.28" rot="R270"/>
+<instance part="R6" gate="G$1" x="45.72" y="81.28" rot="R270"/>
+<instance part="R8" gate="G$1" x="55.88" y="81.28" rot="R270"/>
+<instance part="R9" gate="G$1" x="66.04" y="81.28" rot="R270"/>
+<instance part="KEYPAD" gate="A" x="17.78" y="101.6"/>
+<instance part="CONTROL" gate="A" x="17.78" y="20.32" smashed="yes" rot="R180">
+<attribute name="NAME" x="20.066" y="30.861" size="1.778" layer="95" rot="R180"/>
+<attribute name="VALUE" x="24.13" y="30.48" size="1.778" layer="96" rot="R180"/>
+</instance>
 </instances>
 <busses>
@@
 </segment>
 </net>
-<net name="ROW1" class="0">
-<segment>
-<pinref part="U1" gate="A" pin="PD5"/>
-<wire x1="198.12" y1="76.2" x2="203.2" y2="76.2" width="0.1524" layer="91"/>
-<label x="203.2" y="76.2" size="1.27" layer="95" xref="yes"/>
-</segment>
-<segment>
-<pinref part="KEYPAD" gate="A" pin="1"/>
-<wire x1="50.8" y1="81.28" x2="43.18" y2="81.28" width="0.1524" layer="91"/>
-<label x="43.18" y="81.28" size="1.27" layer="95" rot="MR0" xref="yes"/>
-</segment>
-</net>
-<net name="ROW2" class="0">
-<segment>
-<pinref part="U1" gate="A" pin="PD6"/>
-<wire x1="198.12" y1="73.66" x2="203.2" y2="73.66" width="0.1524" layer="91"/>
-<label x="203.2" y="73.66" size="1.27" layer="95" xref="yes"/>
-</segment>
-<segment>
-<pinref part="KEYPAD" gate="A" pin="3"/>
-<wire x1="50.8" y1="78.74" x2="43.18" y2="78.74" width="0.1524" layer="91"/>
-<label x="43.18" y="78.74" size="1.27" layer="95" rot="MR0" xref="yes"/>
-</segment>
-</net>
-<net name="ROW3" class="0">
-<segment>
-<pinref part="KEYPAD" gate="A" pin="5"/>
-<wire x1="50.8" y1="76.2" x2="43.18" y2="76.2" width="0.1524" layer="91"/>
-<label x="43.18" y="76.2" size="1.27" layer="95" rot="MR0" xref="yes"/>
-</segment>
-<segment>
-<pinref part="U1" gate="A" pin="PD7"/>
-<wire x1="198.12" y1="71.12" x2="203.2" y2="71.12" width="0.1524" layer="91"/>
-<label x="203.2" y="71.12" size="1.27" layer="95" xref="yes"/>
-</segment>
-</net>
-<net name="COL1" class="0">
-<segment>
-<pinref part="U1" gate="A" pin="PB0"/>
-<wire x1="162.56" y1="86.36" x2="157.48" y2="86.36" width="0.1524" layer="91"/>
-<label x="157.48" y="86.36" size="1.27" layer="95" rot="MR0" xref="yes"/>
-</segment>
-<segment>
-<pinref part="KEYPAD" gate="A" pin="2"/>
-<wire x1="58.42" y1="81.28" x2="66.04" y2="81.28" width="0.1524" layer="91"/>
-<label x="66.04" y="81.28" size="1.27" layer="95" xref="yes"/>
-</segment>
-</net>
-<net name="COL2" class="0">
-<segment>
-<pinref part="U1" gate="A" pin="PB1"/>
-<wire x1="162.56" y1="83.82" x2="157.48" y2="83.82" width="0.1524" layer="91"/>
-<label x="157.48" y="83.82" size="1.27" layer="95" rot="MR0" xref="yes"/>
-</segment>
-<segment>
-<pinref part="KEYPAD" gate="A" pin="4"/>
-<wire x1="58.42" y1="78.74" x2="66.04" y2="78.74" width="0.1524" layer="91"/>
-<label x="66.04" y="78.74" size="1.27" layer="95" xref="yes"/>
-</segment>
-</net>
-<net name="COL3" class="0">
-<segment>
-<pinref part="U1" gate="A" pin="PB2"/>
-<wire x1="162.56" y1="81.28" x2="157.48" y2="81.28" width="0.1524" layer="91"/>
-<label x="157.48" y="81.28" size="1.27" layer="95" rot="MR0" xref="yes"/>
-</segment>
-<segment>
-<pinref part="KEYPAD" gate="A" pin="6"/>
-<wire x1="58.42" y1="76.2" x2="66.04" y2="76.2" width="0.1524" layer="91"/>
-<label x="66.04" y="76.2" size="1.27" layer="95" xref="yes"/>
-</segment>
-</net>
 <net name="SERVO" class="0">
 <segment>
@@
 <label x="43.18" y="55.88" size="1.27" layer="95" rot="MR0" xref="yes"/>
 </segment>
-<segment>
-<pinref part="U1" gate="A" pin="ADC6"/>
-<wire x1="162.56" y1="99.06" x2="157.48" y2="99.06" width="0.1524" layer="91"/>
-<label x="157.48" y="99.06" size="1.27" layer="95" rot="MR0" xref="yes"/>
-</segment>
 </net>
 <net name="SOLENOID-SIG" class="0">
@@
 <net name="LED-GRN" class="0">
 <segment>
-<pinref part="U1" gate="A" pin="PC0"/>
-<wire x1="198.12" y1="109.22" x2="203.2" y2="109.22" width="0.1524" layer="91"/>
-<label x="203.2" y="109.22" size="1.27" layer="95" xref="yes"/>
-</segment>
-<segment>
 <pinref part="LOCK-CTRL" gate="A" pin="7"/>
 <wire x1="50.8" y1="48.26" x2="43.18" y2="48.26" width="0.1524" layer="91"/>
@@
 </net>
 <net name="LED-RED" class="0">
-<segment>
-<pinref part="U1" gate="A" pin="PC1"/>
-<wire x1="198.12" y1="106.68" x2="203.2" y2="106.68" width="0.1524" layer="91"/>
-<label x="203.2" y="106.68" size="1.27" layer="95" xref="yes"/>
-</segment>
 <segment>
 <pinref part="LOCK-CTRL" gate="A" pin="8"/>
@@
 <wire x1="50.8" y1="101.6" x2="43.18" y2="101.6" width="0.1524" layer="91"/>
 <wire x1="43.18" y1="101.6" x2="43.18" y2="96.52" width="0.1524" layer="91"/>
-<pinref part="GND12" gate="1" pin="GND"/>
+<pinref part="GND3" gate="1" pin="GND"/>
 </segment>
 </net>
@@
 </segment>
 </net>
+<net name="N$6" class="0">
+<segment>
+<pinref part="U1" gate="A" pin="PD5"/>
+<wire x1="198.12" y1="76.2" x2="203.2" y2="76.2" width="0.1524" layer="91"/>
+<label x="203.2" y="76.2" size="1.778" layer="95"/>
+</segment>
+</net>
+<net name="N$9" class="0">
+<segment>
+<pinref part="U1" gate="A" pin="PD6"/>
+<wire x1="198.12" y1="73.66" x2="203.2" y2="73.66" width="0.1524" layer="91"/>
+<label x="203.2" y="73.66" size="1.778" layer="95"/>
+</segment>
+</net>
+<net name="N$10" class="0">
+<segment>
+<pinref part="U1" gate="A" pin="PD7"/>
+<wire x1="198.12" y1="71.12" x2="203.2" y2="71.12" width="0.1524" layer="91"/>
+<label x="203.2" y="71.12" size="1.778" layer="95"/>
+</segment>
+</net>
+<net name="N$11" class="0">
+<segment>
+<pinref part="U1" gate="A" pin="PB0"/>
+<wire x1="162.56" y1="86.36" x2="157.48" y2="86.36" width="0.1524" layer="91"/>
+<label x="157.48" y="86.36" size="1.778" layer="95"/>
+</segment>
+</net>
+<net name="N$12" class="0">
+<segment>
+<pinref part="U1" gate="A" pin="PB1"/>
+<wire x1="162.56" y1="83.82" x2="157.48" y2="83.82" width="0.1524" layer="91"/>
+<label x="157.48" y="83.82" size="1.778" layer="95"/>
+</segment>
+</net>
+<net name="N$13" class="0">
+<segment>
+<pinref part="U1" gate="A" pin="PB2"/>
+<wire x1="162.56" y1="81.28" x2="157.48" y2="81.28" width="0.1524" layer="91"/>
+<label x="157.48" y="81.28" size="1.778" layer="95"/>
+</segment>
+</net>
+<net name="N$14" class="0">
+<segment>
+<pinref part="U1" gate="A" pin="PC3"/>
+<wire x1="198.12" y1="101.6" x2="203.2" y2="101.6" width="0.1524" layer="91"/>
+<label x="203.2" y="101.6" size="1.778" layer="95"/>
+</segment>
+</net>

Commit message: schematic
Parts:
- R1: value 1K -> 10K
Changed lines of the file:
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@@
 <part name="Q1" library="murata-filter" deviceset="CSTCR" device="" technology="6M00G53Z"/>
 <part name="U1" library="Ava" deviceset="ATMEGA328P-AU" device=""/>
-<part name="R1" library="resistor" deviceset="R-EU_" device="R0805" value="1K"/>
+<part name="R1" library="resistor" deviceset="R-EU_" device="R0805" value="10K"/>
 <part name="C2" library="resistor" deviceset="C-US" device="C1206" value="10uf"/>
 <part name="C4" library="resistor" deviceset="C-EU" device="C0805" value="0.1uF"/>
