File: eagle/keepuntil-v1.0/KeepUntil-v1.0.brd (EAGLE design)
At the start: 100 x 80 mm, 22 parts, among them IC2 REG1117, Q1 CSTCR6M00G53Z, T1 BC846, U1 ATMEGA328P-AU, X1 MINI-USB-32005-201

Commit message: schematic & board
Parts:
- removed JP2: (no value), pinhead:2X04
- added KEYPAD: (no value), pinhead:2X04
- moved R6 74.7 mm to (27.9, 27.9), turned to 270 degrees
- moved R4 67.8 mm to (17.8, 31.8), turned to 90 degrees
- moved R3 62.0 mm to (17.8, 35.6), turned to 270 degrees
- moved R5 41.7 mm to (17.8, 27.9), turned to 90 degrees
- moved R8 2.84 mm to (27.9, 31.8)
- moved R9 2.84 mm to (27.9, 35.6)
Connections:
- removed net COL1: JP2.1
- removed net N$14: U1.26
- removed net N$15: R3.2
- removed net N$16: R4.1
- removed net N$17: R4.2
- removed net N$18: R5.1
- removed net N$19: R6.1
- removed net N$22: R5.2
- removed net N$23: R6.2
- removed net N$5: R3.1
- removed net ROW1: JP2.2, R9.1
- new net KEYPAD: KEYPAD.1, R3.2, R4.2, U1.26
- new net ROW4: KEYPAD.8, R6.2
- net COL2: now also KEYPAD.3, R4.1, R5.2; no longer JP2.3
- net COL3: now also KEYPAD.5, R5.1; no longer JP2.5
- net GND: now also R3.1
- net ROW2: now also KEYPAD.4; no longer JP2.4
- net ROW3: now also KEYPAD.6, R6.1; no longer JP2.6
- net VCC: now also KEYPAD.2, R9.1
Changed lines of the file:
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@@
 <element name="R1" library="resistor" package="R0805" value="10K" x="-38.1" y="46.99"/>
 <element name="R2" library="resistor" package="R0805" value="10K" x="-27.94" y="46.99"/>
-<element name="R3" library="resistor" package="R0805" value="1K" x="-43.18" y="46.99"/>
-<element name="R4" library="resistor" package="R0805" value="1K" x="-48.26" y="46.99"/>
-<element name="R5" library="resistor" package="R0805" value="1K" x="-15.24" y="53.34"/>
-<element name="R6" library="resistor" package="R0805" value="4.7K" x="-45.72" y="40.64"/>
+<element name="R3" library="resistor" package="R0805" value="1K" x="17.78" y="35.56" rot="R270"/>
+<element name="R4" library="resistor" package="R0805" value="1K" x="17.78" y="31.75" rot="R90"/>
+<element name="R5" library="resistor" package="R0805" value="1K" x="17.78" y="27.94" rot="R90"/>
+<element name="R6" library="resistor" package="R0805" value="4.7K" x="27.94" y="27.94" rot="R270"/>
 <element name="R7" library="resistor" package="R0805" value="330" x="-33.02" y="46.99"/>
-<element name="R8" library="resistor" package="R0805" value="4.7K" x="26.67" y="29.21" rot="R270"/>
-<element name="R9" library="resistor" package="R0805" value="4.7K" x="26.67" y="33.02" rot="R270"/>
+<element name="R8" library="resistor" package="R0805" value="4.7K" x="27.94" y="31.75" rot="R270"/>
+<element name="R9" library="resistor" package="R0805" value="4.7K" x="27.94" y="35.56" rot="R270"/>
 <element name="T1" library="transistor" package="SOT23" value="BC846" x="-44.45" y="33.02"/>
 <element name="U1" library="Ava" package="QFP80P900X900X120-32N" value="ATMEGA328P-AU" x="-24.13" y="8.89">
@@
 </element>
 <element name="JP1" library="pinhead" package="2X06" value="" x="-54.61" y="-12.7"/>
-<element name="JP2" library="pinhead" package="2X04" value="" x="22.86" y="30.48" rot="R270"/>
+<element name="KEYPAD" library="pinhead" package="2X04" value="" x="22.86" y="31.75" rot="R270"/>
 </elements>
 <signals>
@@
 <contactref element="C2" pad="1"/>
 <contactref element="R7" pad="2"/>
-<wire x1="-32.07" y1="46.99" x2="-22.99" y2="46.99" width="0" layer="19" extent="1-1"/>
-<wire x1="-37.15" y1="46.99" x2="-32.07" y2="46.99" width="0" layer="19" extent="1-1"/>
-<wire x1="-31.75" y1="33.02" x2="-32.07" y2="46.99" width="0" layer="19" extent="1-1"/>
-<wire x1="-17.7546" y1="19.7104" x2="-31.75" y2="33.02" width="0" layer="19" extent="1-1"/>
+<contactref element="KEYPAD" pad="2"/>
+<contactref element="R9" pad="1"/>
+<wire x1="24.13" y1="35.56" x2="27.94" y2="36.51" width="0" layer="19" extent="1-1"/>
+<wire x1="-17.7546" y1="19.7104" x2="24.13" y2="35.56" width="0" layer="19" extent="1-1"/>
 <wire x1="-19.8882" y1="6.8834" x2="-17.7546" y2="19.7104" width="0" layer="19" extent="1-1"/>
 <wire x1="-28.3718" y1="7.6962" x2="-19.8882" y2="6.8834" width="0" layer="19" extent="1-1"/>
 <wire x1="-28.3718" y1="9.2964" x2="-28.3718" y2="7.6962" width="0" layer="19" extent="1-1"/>
+<wire x1="-31.75" y1="33.02" x2="-17.7546" y2="19.7104" width="0" layer="19" extent="1-1"/>
+<wire x1="-32.07" y1="46.99" x2="-31.75" y2="33.02" width="0" layer="19" extent="1-1"/>
+<wire x1="-37.15" y1="46.99" x2="-32.07" y2="46.99" width="0" layer="19" extent="1-1"/>
+<wire x1="-22.99" y1="46.99" x2="-32.07" y2="46.99" width="0" layer="19" extent="1-1"/>
 </signal>
 <signal name="GND">
@@
 <contactref element="X1" pad="5"/>
 <contactref element="S1" pad="1"/>
+<contactref element="R3" pad="1"/>
 <wire x1="-40.18" y1="6.02" x2="-52.68" y2="-3.81" width="0" layer="19" extent="1-1"/>
 <wire x1="-28.3718" y1="8.4836" x2="-40.18" y2="6.02" width="0" layer="19" extent="1-1"/>
@@
 <wire x1="-32.07" y1="40.64" x2="-26.67" y2="33.02" width="0" layer="19" extent="1-1"/>
 <wire x1="-38.42" y1="40.64" x2="-32.07" y2="40.64" width="0" layer="19" extent="1-1"/>
+<wire x1="17.78" y1="36.51" x2="-38.42" y2="40.64" width="0" layer="19" extent="1-1"/>
 <wire x1="-43.5" y1="31.92" x2="-38.42" y2="40.64" width="0" layer="19" extent="1-1"/>
 <wire x1="-29.058" y1="52.07" x2="-32.07" y2="40.64" width="0" layer="19" extent="1-1"/>
@@
 <contactref element="U1" pad="14"/>
 </signal>
-<signal name="N$14">
-<contactref element="U1" pad="26"/>
-</signal>
-<signal name="ROW1">
-<contactref element="R9" pad="1"/>
-<contactref element="JP2" pad="2"/>
-<wire x1="24.13" y1="34.29" x2="26.67" y2="33.97" width="0" layer="19" extent="1-1"/>
-</signal>
 <signal name="ROW2">
 <contactref element="R9" pad="2"/>
 <contactref element="R8" pad="1"/>
-<contactref element="JP2" pad="4"/>
-<wire x1="26.67" y1="30.16" x2="24.13" y2="31.75" width="0" layer="19" extent="1-1"/>
-<wire x1="26.67" y1="32.07" x2="26.67" y2="30.16" width="0" layer="19" extent="1-1"/>
+<contactref element="KEYPAD" pad="4"/>
+<wire x1="27.94" y1="32.7" x2="24.13" y2="33.02" width="0" layer="19" extent="1-1"/>
+<wire x1="27.94" y1="34.61" x2="27.94" y2="32.7" width="0" layer="19" extent="1-1"/>
 </signal>
 <signal name="ROW3">
 <contactref element="R8" pad="2"/>
-<contactref element="JP2" pad="6"/>
-<wire x1="26.67" y1="28.26" x2="24.13" y2="29.21" width="0" layer="19" extent="1-1"/>
-</signal>
-<signal name="N$5">
-<contactref element="R3" pad="1"/>
-</signal>
-<signal name="N$15">
+<contactref element="KEYPAD" pad="6"/>
+<contactref element="R6" pad="1"/>
+<wire x1="24.13" y1="30.48" x2="27.94" y2="30.8" width="0" layer="19" extent="1-1"/>
+<wire x1="27.94" y1="28.89" x2="24.13" y2="30.48" width="0" layer="19" extent="1-1"/>
+</signal>
+<signal name="COL2">
+<contactref element="KEYPAD" pad="3"/>
+<contactref element="R5" pad="2"/>
+<contactref element="R4" pad="1"/>
+<wire x1="17.78" y1="28.89" x2="21.59" y2="33.02" width="0" layer="19" extent="1-1"/>
+<wire x1="17.78" y1="30.8" x2="17.78" y2="28.89" width="0" layer="19" extent="1-1"/>
+</signal>
+<signal name="COL3">
+<contactref element="KEYPAD" pad="5"/>
+<contactref element="R5" pad="1"/>
+<wire x1="17.78" y1="26.99" x2="21.59" y2="30.48" width="0" layer="19" extent="1-1"/>
+</signal>
+<signal name="ROW4">
+<contactref element="KEYPAD" pad="8"/>
+<contactref element="R6" pad="2"/>
+<wire x1="27.94" y1="26.99" x2="24.13" y2="27.94" width="0" layer="19" extent="1-1"/>
+</signal>
+<signal name="KEYPAD">
+<contactref element="KEYPAD" pad="1"/>
 <contactref element="R3" pad="2"/>
-</signal>
-<signal name="N$16">
-<contactref element="R4" pad="1"/>
-</signal>
-<signal name="N$17">
 <contactref element="R4" pad="2"/>
-</signal>
-<signal name="N$18">
-<contactref element="R5" pad="1"/>
-</signal>
-<signal name="N$19">
-<contactref element="R6" pad="1"/>
-</signal>
-<signal name="N$22">
-<contactref element="R5" pad="2"/>
-</signal>
-<signal name="N$23">
-<contactref element="R6" pad="2"/>
-</signal>
-<signal name="COL1">
-<contactref element="JP2" pad="1"/>
-</signal>
-<signal name="COL2">
-<contactref element="JP2" pad="3"/>
-</signal>
-<signal name="COL3">
-<contactref element="JP2" pad="5"/>
+<contactref element="U1" pad="26"/>
+<wire x1="17.78" y1="34.61" x2="21.59" y2="35.56" width="0" layer="19" extent="1-1"/>
+<wire x1="17.78" y1="32.7" x2="17.78" y2="34.61" width="0" layer="19" extent="1-1"/>
+<wire x1="-22.1234" y1="13.1318" x2="17.78" y2="32.7" width="0" layer="19" extent="1-1"/>
 </signal>
 </signals>

Commit message: schematic
Parts:
- removed R3, R4, R5: 1K, resistor:R0805
- removed R6, R8, R9: 4.7K, resistor:R0805
- added JP2: (no value), pinhead:1X03
- JP1: device pinhead:2X06 -> pinhead:2X11
- moved JP1 15.2 mm to (-39.4, -12.7)
Connections:
- net RTC-SCL renamed SCL
- net RTC-SDA renamed SDA
- removed net KEYPAD: KEYPAD.1, R3.2, R4.2, U1.26
- new net COL1: KEYPAD.1
- new net N$14: U1.24
- new net N$15: U1.25
- new net N$16: U1.26
- new net N$5: U1.23
- new net ROW1: KEYPAD.2
- net COL2: no longer R4.1, R5.2
- net COL3: no longer R5.1
- net GND: now also Q1.2; no longer R3.1
- net ROW2: no longer R8.1, R9.2
- net ROW3: no longer R6.1, R8.2
- net ROW4: no longer R6.2
- net VCC: no longer KEYPAD.2, R9.1
Changed lines of the file:
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@@
 <element name="R1" library="resistor" package="R0805" value="10K" x="-38.1" y="46.99"/>
 <element name="R2" library="resistor" package="R0805" value="10K" x="-27.94" y="46.99"/>
-<element name="R3" library="resistor" package="R0805" value="1K" x="17.78" y="35.56" rot="R270"/>
-<element name="R4" library="resistor" package="R0805" value="1K" x="17.78" y="31.75" rot="R90"/>
-<element name="R5" library="resistor" package="R0805" value="1K" x="17.78" y="27.94" rot="R90"/>
-<element name="R6" library="resistor" package="R0805" value="4.7K" x="27.94" y="27.94" rot="R270"/>
 <element name="R7" library="resistor" package="R0805" value="330" x="-33.02" y="46.99"/>
-<element name="R8" library="resistor" package="R0805" value="4.7K" x="27.94" y="31.75" rot="R270"/>
-<element name="R9" library="resistor" package="R0805" value="4.7K" x="27.94" y="35.56" rot="R270"/>
 <element name="T1" library="transistor" package="SOT23" value="BC846" x="-44.45" y="33.02"/>
 <element name="U1" library="Ava" package="QFP80P900X900X120-32N" value="ATMEGA328P-AU" x="-24.13" y="8.89">
@@
 <attribute name="PROD_ID" value="SWCH-00815" x="-49.53" y="-3.81" size="1.778" layer="27" display="off"/>
 </element>
-<element name="JP1" library="pinhead" package="2X06" value="" x="-54.61" y="-12.7"/>
 <element name="KEYPAD" library="pinhead" package="2X04" value="" x="22.86" y="31.75" rot="R270"/>
+<element name="JP1" library="pinhead" package="2X11" value="" x="-39.37" y="-12.7"/>
+<element name="JP2" library="pinhead" package="1X03" value="" x="-49.53" y="-19.05"/>
 </elements>
 <signals>
@@
 <wire x1="-29.21" y1="30.48" x2="-19.8882" y2="6.096" width="0" layer="19" extent="1-1"/>
 </signal>
-<signal name="RTC-SCL">
+<signal name="SCL">
 <contactref element="U1" pad="28"/>
 </signal>
@@
 <contactref element="T1" pad="3"/>
 </signal>
-<signal name="RTC-SDA">
+<signal name="SDA">
 <contactref element="U1" pad="27"/>
 </signal>
@@
 <contactref element="C2" pad="1"/>
 <contactref element="R7" pad="2"/>
-<contactref element="KEYPAD" pad="2"/>
-<contactref element="R9" pad="1"/>
-<wire x1="24.13" y1="35.56" x2="27.94" y2="36.51" width="0" layer="19" extent="1-1"/>
-<wire x1="-17.7546" y1="19.7104" x2="24.13" y2="35.56" width="0" layer="19" extent="1-1"/>
+<wire x1="-32.07" y1="46.99" x2="-22.99" y2="46.99" width="0" layer="19" extent="1-1"/>
+<wire x1="-37.15" y1="46.99" x2="-32.07" y2="46.99" width="0" layer="19" extent="1-1"/>
+<wire x1="-31.75" y1="33.02" x2="-32.07" y2="46.99" width="0" layer="19" extent="1-1"/>
+<wire x1="-17.7546" y1="19.7104" x2="-31.75" y2="33.02" width="0" layer="19" extent="1-1"/>
 <wire x1="-19.8882" y1="6.8834" x2="-17.7546" y2="19.7104" width="0" layer="19" extent="1-1"/>
 <wire x1="-28.3718" y1="7.6962" x2="-19.8882" y2="6.8834" width="0" layer="19" extent="1-1"/>
 <wire x1="-28.3718" y1="9.2964" x2="-28.3718" y2="7.6962" width="0" layer="19" extent="1-1"/>
-<wire x1="-31.75" y1="33.02" x2="-17.7546" y2="19.7104" width="0" layer="19" extent="1-1"/>
-<wire x1="-32.07" y1="46.99" x2="-31.75" y2="33.02" width="0" layer="19" extent="1-1"/>
-<wire x1="-37.15" y1="46.99" x2="-32.07" y2="46.99" width="0" layer="19" extent="1-1"/>
-<wire x1="-22.99" y1="46.99" x2="-32.07" y2="46.99" width="0" layer="19" extent="1-1"/>
 </signal>
 <signal name="GND">
@@
 <contactref element="X1" pad="5"/>
 <contactref element="S1" pad="1"/>
-<contactref element="R3" pad="1"/>
+<contactref element="Q1" pad="2"/>
 <wire x1="-40.18" y1="6.02" x2="-52.68" y2="-3.81" width="0" layer="19" extent="1-1"/>
 <wire x1="-28.3718" y1="8.4836" x2="-40.18" y2="6.02" width="0" layer="19" extent="1-1"/>
@@
 <wire x1="-20.0406" y1="19.7104" x2="-19.8882" y2="9.2964" width="0" layer="19" extent="1-1"/>
 <wire x1="-26.67" y1="33.02" x2="-20.0406" y2="19.7104" width="0" layer="19" extent="1-1"/>
-<wire x1="-32.07" y1="40.64" x2="-26.67" y2="33.02" width="0" layer="19" extent="1-1"/>
+<wire x1="-25.4" y1="40.64" x2="-26.67" y2="33.02" width="0" layer="19" extent="1-1"/>
+<wire x1="-32.07" y1="40.64" x2="-25.4" y2="40.64" width="0" layer="19" extent="1-1"/>
 <wire x1="-38.42" y1="40.64" x2="-32.07" y2="40.64" width="0" layer="19" extent="1-1"/>
-<wire x1="17.78" y1="36.51" x2="-38.42" y2="40.64" width="0" layer="19" extent="1-1"/>
+<wire x1="-20.19" y1="46.99" x2="-25.4" y2="40.64" width="0" layer="19" extent="1-1"/>
 <wire x1="-43.5" y1="31.92" x2="-38.42" y2="40.64" width="0" layer="19" extent="1-1"/>
-<wire x1="-29.058" y1="52.07" x2="-32.07" y2="40.64" width="0" layer="19" extent="1-1"/>
-<wire x1="-20.19" y1="46.99" x2="-29.058" y2="52.07" width="0" layer="19" extent="1-1"/>
+<wire x1="-29.058" y1="52.07" x2="-20.19" y2="46.99" width="0" layer="19" extent="1-1"/>
 </signal>
 <signal name="N$4">
@@
 </signal>
 <signal name="ROW2">
-<contactref element="R9" pad="2"/>
-<contactref element="R8" pad="1"/>
 <contactref element="KEYPAD" pad="4"/>
-<wire x1="27.94" y1="32.7" x2="24.13" y2="33.02" width="0" layer="19" extent="1-1"/>
-<wire x1="27.94" y1="34.61" x2="27.94" y2="32.7" width="0" layer="19" extent="1-1"/>
 </signal>
 <signal name="ROW3">
-<contactref element="R8" pad="2"/>
 <contactref element="KEYPAD" pad="6"/>
-<contactref element="R6" pad="1"/>
-<wire x1="24.13" y1="30.48" x2="27.94" y2="30.8" width="0" layer="19" extent="1-1"/>
-<wire x1="27.94" y1="28.89" x2="24.13" y2="30.48" width="0" layer="19" extent="1-1"/>
 </signal>
 <signal name="COL2">
 <contactref element="KEYPAD" pad="3"/>
-<contactref element="R5" pad="2"/>
-<contactref element="R4" pad="1"/>
-<wire x1="17.78" y1="28.89" x2="21.59" y2="33.02" width="0" layer="19" extent="1-1"/>
-<wire x1="17.78" y1="30.8" x2="17.78" y2="28.89" width="0" layer="19" extent="1-1"/>
 </signal>
 <signal name="COL3">
 <contactref element="KEYPAD" pad="5"/>
-<contactref element="R5" pad="1"/>
-<wire x1="17.78" y1="26.99" x2="21.59" y2="30.48" width="0" layer="19" extent="1-1"/>
 </signal>
 <signal name="ROW4">
 <contactref element="KEYPAD" pad="8"/>
-<contactref element="R6" pad="2"/>
-<wire x1="27.94" y1="26.99" x2="24.13" y2="27.94" width="0" layer="19" extent="1-1"/>
 </signal>
-<signal name="KEYPAD">
+<signal name="ROW1">
+<contactref element="KEYPAD" pad="2"/>
+</signal>
+<signal name="COL1">
 <contactref element="KEYPAD" pad="1"/>
-<contactref element="R3" pad="2"/>
-<contactref element="R4" pad="2"/>
+</signal>
+<signal name="N$5">
+<contactref element="U1" pad="23"/>
+</signal>
+<signal name="N$14">
+<contactref element="U1" pad="24"/>
+</signal>
+<signal name="N$15">
+<contactref element="U1" pad="25"/>
+</signal>
+<signal name="N$16">
 <contactref element="U1" pad="26"/>
-<wire x1="17.78" y1="34.61" x2="21.59" y2="35.56" width="0" layer="19" extent="1-1"/>
-<wire x1="17.78" y1="32.7" x2="17.78" y2="34.61" width="0" layer="19" extent="1-1"/>
-<wire x1="-22.1234" y1="13.1318" x2="17.78" y2="32.7" width="0" layer="19" extent="1-1"/>
 </signal>
 </signals>

Commit message: Schematic
Parts:
- removed JP2: (no value), pinhead:1X03
- removed X1: MINI-USB-32005-201, con-cypressindustries:32005-201
- added C1: 0.1uF, resistor:C0805
- added J1: USB-MICROB, SparkFun-Connectors:USB-MICROB
- added SERIAL: (no value), pinhead:1X06
Connections:
- new net N$17: C1.2, SERIAL.6
- net GND: now also J1.GND, J1.MT1, J1.MT2, SERIAL.1; no longer X1.5
- net N$4: now also J1.VBUS; no longer X1.1
- net RESET: now also C1.1
- net RX: now also SERIAL.4
- net TX: now also SERIAL.5
- net VCC: now also SERIAL.3
Changed lines of the file:
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@@
 <attribute name="OC_NEWARK" value="14R4631" x="-24.13" y="8.89" size="1.778" layer="27" display="off"/>
-</element>
-<element name="X1" library="con-cypressindustries" package="32005-201" value="MINI-USB-32005-201" x="-43.18" y="7.62">
-<attribute name="OC_FARNELL" value="unknown" x="-43.18" y="7.62" size="1.778" layer="27" display="off"/>
-<attribute name="MF" value="" x="-43.18" y="7.62" size="1.778" layer="27" display="off"/>
-<attribute name="MPN" value="" x="-43.18" y="7.62" size="1.778" layer="27" display="off"/>
-<attribute name="OC_NEWARK" value="unknown" x="-43.18" y="7.62" size="1.778" layer="27" display="off"/>
 </element>
 <element name="S1" library="SparkFun-Electromechanical" package="TACTILE-SWITCH-1101NE" value="SWITCH-MOMENTARY-2SMD-1101NE" x="-49.53" y="-3.81">
@@
 <element name="KEYPAD" library="pinhead" package="2X04" value="" x="22.86" y="31.75" rot="R270"/>
 <element name="JP1" library="pinhead" package="2X11" value="" x="-39.37" y="-12.7"/>
-<element name="JP2" library="pinhead" package="1X03" value="" x="-49.53" y="-19.05"/>
+<element name="SERIAL" library="pinhead" package="1X06" value="" x="-45.72" y="-19.05"/>
+<element name="C1" library="resistor" package="C0805" value="0.1uF" x="-50.8" y="-24.13"/>
+<element name="J1" library="SparkFun-Connectors" package="USB-MICROB" value="USB-MICROB" x="-48.26" y="-31.75">
+<attribute name="PROD_ID" value="CONN-09505" x="-48.26" y="-31.75" size="1.778" layer="27" display="off"/>
+</element>
 </elements>
 <signals>
@@
 <contactref element="ISP" pad="4"/>
 <contactref element="S1" pad="2"/>
+<contactref element="C1" pad="1"/>
+<wire x1="-46.38" y1="-3.81" x2="-51.75" y2="-24.13" width="0" layer="19" extent="1-1"/>
 <wire x1="-24.5364" y1="13.1318" x2="-46.38" y2="-3.81" width="0" layer="19" extent="1-1"/>
 <wire x1="-29.21" y1="33.02" x2="-24.5364" y2="13.1318" width="0" layer="19" extent="1-1"/>
@@
 <signal name="TX">
 <contactref element="U1" pad="31"/>
+<contactref element="SERIAL" pad="5"/>
+<wire x1="-26.1366" y1="13.1318" x2="-41.91" y2="-19.05" width="0" layer="19" extent="1-1"/>
 </signal>
 <signal name="RX">
 <contactref element="U1" pad="30"/>
+<contactref element="SERIAL" pad="4"/>
+<wire x1="-25.3238" y1="13.1318" x2="-44.45" y2="-19.05" width="0" layer="19" extent="1-1"/>
 </signal>
 <signal name="SOLENOID-SIG">
@@
 <contactref element="C2" pad="1"/>
 <contactref element="R7" pad="2"/>
-<wire x1="-32.07" y1="46.99" x2="-22.99" y2="46.99" width="0" layer="19" extent="1-1"/>
+<contactref element="SERIAL" pad="3"/>
+<wire x1="-28.3718" y1="7.6962" x2="-46.99" y2="-19.05" width="0" layer="19" extent="1-1"/>
+<wire x1="-28.3718" y1="9.2964" x2="-28.3718" y2="7.6962" width="0" layer="19" extent="1-1"/>
+<wire x1="-19.8882" y1="6.8834" x2="-28.3718" y2="7.6962" width="0" layer="19" extent="1-1"/>
+<wire x1="-17.7546" y1="19.7104" x2="-19.8882" y2="6.8834" width="0" layer="19" extent="1-1"/>
+<wire x1="-31.75" y1="33.02" x2="-17.7546" y2="19.7104" width="0" layer="19" extent="1-1"/>
+<wire x1="-32.07" y1="46.99" x2="-31.75" y2="33.02" width="0" layer="19" extent="1-1"/>
 <wire x1="-37.15" y1="46.99" x2="-32.07" y2="46.99" width="0" layer="19" extent="1-1"/>
-<wire x1="-31.75" y1="33.02" x2="-32.07" y2="46.99" width="0" layer="19" extent="1-1"/>
-<wire x1="-17.7546" y1="19.7104" x2="-31.75" y2="33.02" width="0" layer="19" extent="1-1"/>
-<wire x1="-19.8882" y1="6.8834" x2="-17.7546" y2="19.7104" width="0" layer="19" extent="1-1"/>
-<wire x1="-28.3718" y1="7.6962" x2="-19.8882" y2="6.8834" width="0" layer="19" extent="1-1"/>
-<wire x1="-28.3718" y1="9.2964" x2="-28.3718" y2="7.6962" width="0" layer="19" extent="1-1"/>
+<wire x1="-22.99" y1="46.99" x2="-32.07" y2="46.99" width="0" layer="19" extent="1-1"/>
 </signal>
 <signal name="GND">
@@
 <contactref element="T1" pad="2"/>
 <contactref element="ISP" pad="6"/>
-<contactref element="X1" pad="5"/>
 <contactref element="S1" pad="1"/>
 <contactref element="Q1" pad="2"/>
-<wire x1="-40.18" y1="6.02" x2="-52.68" y2="-3.81" width="0" layer="19" extent="1-1"/>
-<wire x1="-28.3718" y1="8.4836" x2="-40.18" y2="6.02" width="0" layer="19" extent="1-1"/>
+<contactref element="SERIAL" pad="1"/>
+<contactref element="J1" pad="MT2"/>
+<contactref element="J1" pad="GND"/>
+<contactref element="J1" pad="MT1"/>
+<wire x1="-46.96" y1="-29.1" x2="-52.26" y2="-31.75" width="0" layer="19" extent="1-1"/>
+<wire x1="-44.26" y1="-31.75" x2="-46.96" y2="-29.1" width="0" layer="19" extent="1-1"/>
+<wire x1="-52.07" y1="-19.05" x2="-46.96" y2="-29.1" width="0" layer="19" extent="1-1"/>
+<wire x1="-52.68" y1="-3.81" x2="-52.07" y2="-19.05" width="0" layer="19" extent="1-1"/>
+<wire x1="-28.3718" y1="8.4836" x2="-52.68" y2="-3.81" width="0" layer="19" extent="1-1"/>
 <wire x1="-28.3718" y1="10.0838" x2="-28.3718" y2="8.4836" width="0" layer="19" extent="1-1"/>
 <wire x1="-19.8882" y1="9.2964" x2="-28.3718" y2="8.4836" width="0" layer="19" extent="1-1"/>
@@
 <signal name="N$4">
 <contactref element="IC2" pad="3"/>
-<contactref element="X1" pad="1"/>
 <contactref element="C4" pad="1"/>
-<wire x1="-15.4686" y1="19.7104" x2="-40.18" y2="9.22" width="0" layer="19" extent="1-1"/>
+<contactref element="J1" pad="VBUS"/>
+<wire x1="-15.4686" y1="19.7104" x2="-49.56" y2="-29.1" width="0" layer="19" extent="1-1"/>
 <wire x1="-33.97" y1="40.64" x2="-15.4686" y2="19.7104" width="0" layer="19" extent="1-1"/>
 </signal>
@@
 <contactref element="U1" pad="26"/>
 </signal>
+<signal name="N$17">
+<contactref element="SERIAL" pad="6"/>
+<contactref element="C1" pad="2"/>
+<wire x1="-39.37" y1="-19.05" x2="-49.85" y2="-24.13" width="0" layer="19" extent="1-1"/>
+</signal>
 </signals>

Commit message: schematic
Parts:
- removed JP1: (no value), pinhead:2X11
Changed lines of the file:
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@@
 </element>
 <element name="KEYPAD" library="pinhead" package="2X04" value="" x="22.86" y="31.75" rot="R270"/>
-<element name="JP1" library="pinhead" package="2X11" value="" x="-39.37" y="-12.7"/>
 <element name="SERIAL" library="pinhead" package="1X06" value="" x="-45.72" y="-19.05"/>
 <element name="C1" library="resistor" package="C0805" value="0.1uF" x="-50.8" y="-24.13"/>
