File: eagle/keepuntil-v1.0/KeepUntil-v1.0.0.sch (EAGLE design)
At the start: 16 parts, among them IC2 REG1117, J1 USB-MICROB, Q1 CSTCR6M00G53Z, T1 BC846, U1 ATMEGA328P-AU

Commit message: board
Connections:
- net SOLENOID-SIG: no longer U1.PD2
Changed lines of the file:
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@@
 <net name="SOLENOID-SIG" class="0">
-<segment>
-<pinref part="U1" gate="A" pin="PD2"/>
-<wire x1="198.12" y1="91.44" x2="203.2" y2="91.44" width="0.1524" layer="91"/>
-</segment>
 <segment>
 <pinref part="R2" gate="G$1" pin="2"/>
