File: eagle/keepuntil-v1.0/KeepUntil-v1.0.1.brd (EAGLE design)
At the start: 32 x 40 mm, 16 parts, among them IC2 REG1117, J1 USB-MICROB, Q1 CSTCR6M00G53Z, T1 BC846, U1 ATMEGA328P-AU

Commit message: board
Connections:
- net SOLENOID-SIG: no longer JP1.6
Routing:
- net VCC: track 112.3 -> 75.3 mm
- net GND: track 78.3 -> 47.6 mm, vias 3 -> 4
- net RX: track 32.4 -> 12.7 mm, vias 0 -> 1
- net MISO: track 46.0 -> 27.4 mm, vias 0 -> 1
- net RTC-SCL: track 23.4 -> 8.74 mm, vias 1 -> 0
- net SCK: track 30.6 -> 42.1 mm, vias 1 -> 0
- net SOLENOID-SIG: track 45.4 -> 35.6 mm, vias 1 -> 0
- net N$4: track 19.3 -> 27.4 mm
- net RESET: track 59.7 -> 67.7 mm, vias 3 -> 0
- net SOLENOID: track 17.5 -> 20.0 mm
- net N$1: track 9.39 -> 8.21 mm, vias 2 -> 0
Other:
- board text added: "-->"
- board text added: "BTRX/VCC"
- board text added: "BTTX/GND"
- board text added: "NC/VCC"
- board text added: "RTC/GND SCL"
- board text added: "RTC/VCC SDA"
- board text added: "SOL/VCC"
- board text added: "SRVO/GND"
- board text removed: "<--"
- board text removed: "BTRX|+"
- board text removed: "BTTX|-"
- board text removed: "RTCSCL|-"
- board text removed: "RTCSDA|+"
- board text removed: "SOLSIG|+"
- board text removed: "SOL|+"
- board text removed: "SRVO|-"
