File: eagle/keepuntil-v1.0/KeepUntil-v1.0.1.brd (EAGLE design)
At the start: 37 x 45 mm, 18 parts, among them IC2 REG1117, J2 USBSMD, Q1 CSTCR6M00G53Z, T1 BC846, U1 ATMEGA328P-AU

Commit message: testing phonegap
Parts:
- removed ISP: (no value), pinhead:2X03
- added J1: (no value), SparkFun-Connectors:2X3-SHROUDED
- moved BLUETOOTH 19.4 mm to (6.75, 37.6)
- moved RTC 15.0 mm to (28.1, 37.6)
- moved T1 2.18 mm to (14.5, 31.9), turned to 180 degrees
- moved LOCK-CTRL 1.00 mm to (27.6, 29.7)
Connections:
- net BT-RX: now also U1.1; no longer U1.23
- net BT-TX: now also U1.2; no longer U1.24
- net GND: now also J1.6; no longer ISP.6
- net MISO: now also J1.3; no longer ISP.3
- net MOSI: now also J1.5; no longer ISP.5
- net RESET: now also J1.4; no longer ISP.4
- net SCK: now also J1.1; no longer ISP.1
- net VCC: now also J1.2; no longer ISP.2
Routing:
- net GND: track 133.1 -> 77.0 mm, vias 0 -> 2
- net VCC: track 100.8 -> 118.9 mm
- net RX: track 30.6 -> 13.7 mm
- net N$3: track 16.0 -> 7.74 mm
- net MOSI: track 6.53 -> 14.1 mm
- net SOLENOID: track 32.8 -> 40.1 mm
- net MISO: track 4.91 -> 10.6 mm
- net SCK: track 3.90 -> 8.71 mm
- net RESET: track 83.9 -> 79.5 mm
- net RTC-SCL: track 10.6 -> 14.4 mm
- net BT-TX: track 15.6 -> 18.6 mm, vias 1 -> 0
- net N$17: track 31.7 -> 30.4 mm
- net BT-RX: track 12.3 -> 13.2 mm, vias 0 -> 1
- net TX: track 11.1 -> 11.6 mm, vias 1 -> 0
- net RTC-SDA: track 14.5 -> 14.2 mm, vias 0 -> 1
- added copper zone on layer 1, net VCC
Other:
- board text added: "+"
- board text added: "3/5/2016"
- board text added: "BLUETOOTH"
- board text added: "BRIDGETOWN ELECTRONICS"
- board text added: "KeepUntil Box"
- board text added: "NC"
- board text added: "REAL TIME CLOCK"
- board text added: "Rev 1.0"
- board text added: "SERIAL"
- board text removed: "MISO/RST"
- board text removed: "MOSI/GND"
- board text removed: "SCK/VCC"

Commit message: mobile app dev
Parts:
- renumbered J1 to ISP, RTC1 to SERIAL
Changed lines of the file:
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@@
 <attribute name="VALUE" x="23.105" y="33.48" size="1.27" layer="27" rot="R270"/>
 </element>
-<element name="RTC1" library="adafruit" package="1X06-CLEAN" value="" x="6.75" y="27" smashed="yes" rot="R90">
+<element name="SERIAL" library="adafruit" package="1X06-CLEAN" value="" x="6.75" y="27" smashed="yes" rot="R90">
 <attribute name="VALUE" x="9.925" y="19.38" size="1.27" layer="27" rot="R90"/>
 </element>
-<element name="J1" library="SparkFun-Connectors" package="2X3-SHROUDED" value="" x="31.5" y="16.75" smashed="yes">
+<element name="ISP" library="SparkFun-Connectors" package="2X3-SHROUDED" value="" x="31.5" y="16.75" smashed="yes">
 <attribute name="PROD_ID" value="CONN-10681" x="31.5" y="16.75" size="1.778" layer="27" display="off"/>
 <attribute name="VALUE" x="28.579" y="24.624" size="0.4064" layer="27" font="vector"/>
@@
 <contactref element="S1" pad="2"/>
 <contactref element="C1" pad="1"/>
-<contactref element="J1" pad="4"/>
+<contactref element="ISP" pad="4"/>
 <wire x1="9.6012" y1="8.2296" x2="9.6012" y2="10.8204" width="0.1524" layer="1"/>
 <wire x1="9.6012" y1="10.8204" x2="9.51" y2="10.94" width="0.1524" layer="1"/>
@@
 <signal name="MISO">
 <contactref element="U1" pad="16"/>
-<contactref element="J1" pad="3"/>
+<contactref element="ISP" pad="3"/>
 <wire x1="25.2984" y1="21.6408" x2="21.7932" y2="21.6408" width="0.1524" layer="1"/>
 <wire x1="30.1752" y1="16.764" x2="25.2984" y2="21.6408" width="0.1524" layer="1"/>
@@
 <signal name="MOSI">
 <contactref element="U1" pad="15"/>
-<contactref element="J1" pad="5"/>
+<contactref element="ISP" pad="5"/>
 <wire x1="20.8788" y1="19.9644" x2="20.8788" y2="21.6408" width="0.1524" layer="1"/>
 <wire x1="22.7076" y1="18.1356" x2="20.8788" y2="19.9644" width="0.1524" layer="1"/>
@@
 <signal name="SCK">
 <contactref element="U1" pad="17"/>
-<contactref element="J1" pad="1"/>
+<contactref element="ISP" pad="1"/>
 <wire x1="26.5176" y1="23.0124" x2="23.1648" y2="23.0124" width="0.1524" layer="1"/>
 <wire x1="30.1752" y1="19.3548" x2="26.5176" y2="23.0124" width="0.1524" layer="1"/>
@@
 <signal name="TX">
 <contactref element="U1" pad="31"/>
-<contactref element="RTC1" pad="5"/>
+<contactref element="SERIAL" pad="5"/>
 <wire x1="16.764" y1="30.7848" x2="16.764" y2="30.1752" width="0.1524" layer="1"/>
 <wire x1="15.6972" y1="31.8516" x2="16.764" y2="30.7848" width="0.1524" layer="1"/>
@@
 <signal name="RX">
 <contactref element="U1" pad="30"/>
-<contactref element="RTC1" pad="4"/>
+<contactref element="SERIAL" pad="4"/>
 <wire x1="17.526" y1="30.9372" x2="17.526" y2="30.1752" width="0.1524" layer="1"/>
 <wire x1="16.4592" y1="32.004" x2="17.526" y2="30.9372" width="0.1524" layer="1"/>
@@
 <contactref element="LOCK-CTRL" pad="6"/>
 <contactref element="BLUETOOTH" pad="1"/>
-<contactref element="RTC1" pad="3"/>
-<contactref element="J1" pad="2"/>
+<contactref element="SERIAL" pad="3"/>
+<contactref element="ISP" pad="2"/>
 <wire x1="23.622" y1="11.2776" x2="23.622" y2="10.5156" width="0.1524" layer="1"/>
 <wire x1="18.8976" y1="16.002" x2="23.622" y2="11.2776" width="0.1524" layer="1"/>
@@
 <contactref element="LOCK-CTRL" pad="2"/>
 <contactref element="BLUETOOTH" pad="2"/>
-<contactref element="RTC1" pad="1"/>
+<contactref element="SERIAL" pad="1"/>
 <polygon width="0.4064" layer="16">
 <vertex x="0" y="0"/>
@@
 <vertex x="0" y="45"/>
 </polygon>
-<contactref element="J1" pad="6"/>
+<contactref element="ISP" pad="6"/>
 <wire x1="12.4968" y1="14.3256" x2="12.4968" y2="12.954" width="0.1524" layer="1"/>
 <wire x1="13.5636" y1="15.3924" x2="12.4968" y2="14.3256" width="0.1524" layer="1"/>
@@
 <signal name="N$17">
 <contactref element="C1" pad="2"/>
-<contactref element="RTC1" pad="6"/>
+<contactref element="SERIAL" pad="6"/>
 <wire x1="23.622" y1="21.0312" x2="23.622" y2="17.9832" width="0.1524" layer="1"/>
 <wire x1="23.622" y1="22.86" x2="23.622" y2="21.0312" width="0.1524" layer="16"/>
