File: eagle/keepuntil-v1.0/KeepUntil-v1.0.1.sch (EAGLE design)
At the start: 16 parts, among them IC2 REG1117, J1 USB-MICROB, Q1 CSTCR6M00G53Z, T1 BC846, U1 ATMEGA328P-AU

Commit message: board
Connections:
- net SOLENOID-SIG: no longer JP1.6
Changed lines of the file:
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@@
 <label x="203.2" y="111.76" size="1.27" layer="95" xref="yes"/>
-</segment>
-<segment>
-<wire x1="93.98" y1="35.56" x2="101.6" y2="35.56" width="0.1524" layer="91"/>
-<label x="101.6" y="35.56" size="1.27" layer="95" xref="yes"/>
-<pinref part="JP1" gate="A" pin="6"/>
 </segment>
 </net>
