File: eagle/keepuntil-v1.0/KeepUntil-v1.0.1.sch (EAGLE design)
At the start: 16 parts, among them IC2 REG1117, J1 USB-MICROB, Q1 CSTCR6M00G53Z, T1 BC846, U1 ATMEGA328P-AU

Commit message: new board layout
Parts:
- removed J1: USB-MICROB, SparkFun-Connectors:USB-MICROB
- removed JP1: (no value), pinhead:PINHD-2X7
- removed SERIAL: (no value), pinhead:PINHD-1X6
- added BLUETOOTH: 1X4-CLEANBIG, adafruit:1X4-CLEANBIG
- added J2: USBSMD, SparkFun-Connectors:USBSMD
- added LOCK-CTRL: (no value), pinhead:PINHD-2X3
- added RTC, RTC1: (no value), adafruit:PINHD-1X6CLEAN
- C1, C4: value 0.1uF -> .1uF
Connections:
- net SOLENOID-SIG renamed SOL-SIG
- net BT-RX: now also BLUETOOTH.3; no longer JP1.2
- net BT-TX: now also BLUETOOTH.4; no longer JP1.4
- net GND: now also BLUETOOTH.2, J2.GND, LOCK-CTRL.2, RTC.1, RTC1.1; no longer J1.GND, JP1.13, JP1.3, JP1.9, SERIAL.1
- net N$17: now also RTC1.6; no longer SERIAL.6
- net N$4: now also J2.VBUS; no longer J1.VBUS
- net RTC-SCL: now also RTC.4; no longer JP1.14
- net RTC-SDA: now also RTC.3; no longer JP1.12
- net RX: now also RTC1.4; no longer SERIAL.4
- net SERVO: now also LOCK-CTRL.1; no longer JP1.10
- net SOLENOID: now also LOCK-CTRL.5; no longer JP1.8
- net TX: now also RTC1.5; no longer SERIAL.5
- net VCC: now also BLUETOOTH.1, LOCK-CTRL.4, LOCK-CTRL.6, RTC.2, RTC1.3; no longer JP1.1, JP1.11, JP1.5, JP1.7, SERIAL.3
Other:
- moved on the sheet: C1, ISP, R2, T1

Commit message: testing phonegap
Parts:
- removed ISP: (no value), pinhead:PINHD-2X3
- added J1: (no value), SparkFun-Connectors:M03X2SHROUD
Connections:
- net BT-RX: now also U1.PD3; no longer U1.PC0
- net BT-TX: now also U1.PD4; no longer U1.PC1
- net GND: now also J1.6; no longer ISP.6
- net MISO: now also J1.3; no longer ISP.3
- net MOSI: now also J1.5; no longer ISP.5
- net RESET: now also J1.4; no longer ISP.4
- net SCK: now also J1.1; no longer ISP.1
- net VCC: now also J1.2; no longer ISP.2
Changed lines of the file:
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@@
 <part name="LED1" library="led" deviceset="LED" device="SMT1206"/>
 <part name="R7" library="resistor" deviceset="R-EU_" device="R0805" value="330"/>
-<part name="ISP" library="pinhead" deviceset="PINHD-2X3" device=""/>
 <part name="T1" library="transistor" deviceset="BC846" device=""/>
 <part name="R2" library="resistor" deviceset="R-EU_" device="R0805" value="10K"/>
@@
 <part name="LOCK-CTRL" library="pinhead" deviceset="PINHD-2X3" device=""/>
 <part name="RTC1" library="adafruit" deviceset="PINHD-1X6" device="CLEAN"/>
+<part name="J1" library="SparkFun-Connectors" deviceset="M03X2" device="SHROUD"/>
 </parts>
 <sheets>
@@
 <instance part="LED1" gate="G$1" x="93.98" y="132.08"/>
 <instance part="R7" gate="G$1" x="93.98" y="139.7" rot="R90"/>
-<instance part="ISP" gate="A" x="39.116" y="84.836"/>
 <instance part="T1" gate="G$1" x="105.156" y="26.416"/>
 <instance part="R2" gate="G$1" x="94.996" y="26.416" rot="R180"/>
@@
 <instance part="LOCK-CTRL" gate="A" x="73.66" y="50.8"/>
 <instance part="RTC1" gate="A" x="77.216" y="83.82" rot="R180"/>
+<instance part="J1" gate="G$1" x="40.894" y="84.836"/>
 </instances>
 <busses>
@@
 </segment>
 <segment>
-<pinref part="ISP" gate="A" pin="4"/>
-<wire x1="44.196" y1="84.836" x2="51.816" y2="84.836" width="0.1524" layer="91"/>
+<wire x1="44.196" y1="84.836" x2="48.514" y2="84.836" width="0.1524" layer="91"/>
 <label x="51.816" y="84.836" size="1.27" layer="95" xref="yes"/>
+<pinref part="J1" gate="G$1" pin="4"/>
+<wire x1="48.514" y1="84.836" x2="51.816" y2="84.836" width="0.1524" layer="91"/>
+<junction x="48.514" y="84.836"/>
 </segment>
 <segment>
@@
 </segment>
 <segment>
-<pinref part="ISP" gate="A" pin="3"/>
-<wire x1="36.576" y1="84.836" x2="28.956" y2="84.836" width="0.1524" layer="91"/>
+<wire x1="36.576" y1="84.836" x2="33.274" y2="84.836" width="0.1524" layer="91"/>
 <label x="28.956" y="84.836" size="1.27" layer="95" rot="R180" xref="yes"/>
+<pinref part="J1" gate="G$1" pin="3"/>
+<wire x1="33.274" y1="84.836" x2="28.956" y2="84.836" width="0.1524" layer="91"/>
+<junction x="33.274" y="84.836"/>
 </segment>
 </net>
@@
 </segment>
 <segment>
-<pinref part="ISP" gate="A" pin="5"/>
-<wire x1="36.576" y1="82.296" x2="28.956" y2="82.296" width="0.1524" layer="91"/>
+<wire x1="36.576" y1="82.296" x2="33.274" y2="82.296" width="0.1524" layer="91"/>
 <label x="28.956" y="82.296" size="1.27" layer="95" rot="R180" xref="yes"/>
+<pinref part="J1" gate="G$1" pin="5"/>
+<wire x1="33.274" y1="82.296" x2="28.956" y2="82.296" width="0.1524" layer="91"/>
+<junction x="33.274" y="82.296"/>
 </segment>
 </net>
@@
 </segment>
 <segment>
-<pinref part="ISP" gate="A" pin="1"/>
-<wire x1="36.576" y1="87.376" x2="28.956" y2="87.376" width="0.1524" layer="91"/>
+<wire x1="36.576" y1="87.376" x2="33.274" y2="87.376" width="0.1524" layer="91"/>
 <label x="28.956" y="87.376" size="1.27" layer="95" rot="MR0" xref="yes"/>
+<pinref part="J1" gate="G$1" pin="1"/>
+<wire x1="33.274" y1="87.376" x2="28.956" y2="87.376" width="0.1524" layer="91"/>
+<junction x="33.274" y="87.376"/>
 </segment>
 </net>
@@
 </segment>
 <segment>
-<pinref part="ISP" gate="A" pin="2"/>
-<wire x1="44.196" y1="87.376" x2="51.816" y2="87.376" width="0.1524" layer="91"/>
+<wire x1="44.196" y1="87.376" x2="48.514" y2="87.376" width="0.1524" layer="91"/>
+<wire x1="48.514" y1="87.376" x2="51.816" y2="87.376" width="0.1524" layer="91"/>
 <wire x1="51.816" y1="87.376" x2="51.816" y2="92.456" width="0.1524" layer="91"/>
 <pinref part="P+6" gate="VCC" pin="VCC"/>
+<pinref part="J1" gate="G$1" pin="2"/>
+<junction x="48.514" y="87.376"/>
 </segment>
 <segment>
@@
 </segment>
 <segment>
-<pinref part="ISP" gate="A" pin="6"/>
-<wire x1="44.196" y1="82.296" x2="51.816" y2="82.296" width="0.1524" layer="91"/>
+<wire x1="44.196" y1="82.296" x2="48.514" y2="82.296" width="0.1524" layer="91"/>
+<wire x1="48.514" y1="82.296" x2="51.816" y2="82.296" width="0.1524" layer="91"/>
 <wire x1="51.816" y1="82.296" x2="51.816" y2="77.216" width="0.1524" layer="91"/>
 <pinref part="GND7" gate="1" pin="GND"/>
+<pinref part="J1" gate="G$1" pin="6"/>
+<junction x="48.514" y="82.296"/>
 </segment>
 <segment>
@@
 <net name="BT-TX" class="0">
 <segment>
-<pinref part="U1" gate="A" pin="PC1"/>
-<wire x1="208.28" y1="116.84" x2="213.36" y2="116.84" width="0.1524" layer="91"/>
-<label x="213.36" y="116.84" size="1.27" layer="95" xref="yes"/>
-</segment>
-<segment>
 <pinref part="BLUETOOTH" gate="G$1" pin="4"/>
 <wire x1="30.48" y1="48.26" x2="27.94" y2="48.26" width="0.1524" layer="91"/>
 <label x="27.94" y="48.26" size="1.27" layer="95" rot="MR0" xref="yes"/>
 </segment>
+<segment>
+<pinref part="U1" gate="A" pin="PD4"/>
+<wire x1="208.28" y1="88.9" x2="213.36" y2="88.9" width="0.1524" layer="91"/>
+<label x="213.36" y="88.9" size="1.27" layer="95" xref="yes"/>
+</segment>
 </net>
 <net name="BT-RX" class="0">
-<segment>
-<pinref part="U1" gate="A" pin="PC0"/>
-<wire x1="208.28" y1="119.38" x2="213.36" y2="119.38" width="0.1524" layer="91"/>
-<label x="213.36" y="119.38" size="1.27" layer="95" xref="yes"/>
-</segment>
 <segment>
 <pinref part="BLUETOOTH" gate="G$1" pin="3"/>
@@
 <label x="27.94" y="50.8" size="1.27" layer="95" rot="MR0" xref="yes"/>
 </segment>
-</net>
+<segment>
+<pinref part="U1" gate="A" pin="PD3"/>
+<wire x1="208.28" y1="91.44" x2="213.36" y2="91.44" width="0.1524" layer="91"/>
+<label x="213.36" y="91.44" size="1.27" layer="95" xref="yes"/>
+</segment>
+</net>

Commit message: mobile app dev
Parts:
- renumbered J1 to ISP, RTC1 to SERIAL
Changed lines of the file:
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@@
 <part name="BLUETOOTH" library="adafruit" deviceset="1X4" device="-CLEANBIG"/>
 <part name="LOCK-CTRL" library="pinhead" deviceset="PINHD-2X3" device=""/>
-<part name="RTC1" library="adafruit" deviceset="PINHD-1X6" device="CLEAN"/>
-<part name="J1" library="SparkFun-Connectors" deviceset="M03X2" device="SHROUD"/>
+<part name="SERIAL" library="adafruit" deviceset="PINHD-1X6" device="CLEAN"/>
+<part name="ISP" library="SparkFun-Connectors" deviceset="M03X2" device="SHROUD"/>
 </parts>
 <sheets>
@@
 </instance>
 <instance part="LOCK-CTRL" gate="A" x="73.66" y="50.8"/>
-<instance part="RTC1" gate="A" x="77.216" y="83.82" rot="R180"/>
-<instance part="J1" gate="G$1" x="40.894" y="84.836"/>
+<instance part="SERIAL" gate="A" x="77.216" y="83.82" rot="R180"/>
+<instance part="ISP" gate="G$1" x="40.894" y="84.836"/>
 </instances>
 <busses>
@@
 <wire x1="44.196" y1="84.836" x2="48.514" y2="84.836" width="0.1524" layer="91"/>
 <label x="51.816" y="84.836" size="1.27" layer="95" xref="yes"/>
-<pinref part="J1" gate="G$1" pin="4"/>
+<pinref part="ISP" gate="G$1" pin="4"/>
 <wire x1="48.514" y1="84.836" x2="51.816" y2="84.836" width="0.1524" layer="91"/>
 <junction x="48.514" y="84.836"/>
@@
 <wire x1="36.576" y1="84.836" x2="33.274" y2="84.836" width="0.1524" layer="91"/>
 <label x="28.956" y="84.836" size="1.27" layer="95" rot="R180" xref="yes"/>
-<pinref part="J1" gate="G$1" pin="3"/>
+<pinref part="ISP" gate="G$1" pin="3"/>
 <wire x1="33.274" y1="84.836" x2="28.956" y2="84.836" width="0.1524" layer="91"/>
 <junction x="33.274" y="84.836"/>
@@
 <wire x1="36.576" y1="82.296" x2="33.274" y2="82.296" width="0.1524" layer="91"/>
 <label x="28.956" y="82.296" size="1.27" layer="95" rot="R180" xref="yes"/>
-<pinref part="J1" gate="G$1" pin="5"/>
+<pinref part="ISP" gate="G$1" pin="5"/>
 <wire x1="33.274" y1="82.296" x2="28.956" y2="82.296" width="0.1524" layer="91"/>
 <junction x="33.274" y="82.296"/>
@@
 <wire x1="36.576" y1="87.376" x2="33.274" y2="87.376" width="0.1524" layer="91"/>
 <label x="28.956" y="87.376" size="1.27" layer="95" rot="MR0" xref="yes"/>
-<pinref part="J1" gate="G$1" pin="1"/>
+<pinref part="ISP" gate="G$1" pin="1"/>
 <wire x1="33.274" y1="87.376" x2="28.956" y2="87.376" width="0.1524" layer="91"/>
 <junction x="33.274" y="87.376"/>
@@
 <wire x1="79.756" y1="86.36" x2="87.376" y2="86.36" width="0.1524" layer="91"/>
 <label x="87.376" y="86.36" size="1.27" layer="95" rot="MR180" xref="yes"/>
-<pinref part="RTC1" gate="A" pin="5"/>
+<pinref part="SERIAL" gate="A" pin="5"/>
 </segment>
 </net>
@@
 <wire x1="79.756" y1="83.82" x2="87.376" y2="83.82" width="0.1524" layer="91"/>
 <label x="87.376" y="83.82" size="1.27" layer="95" rot="MR180" xref="yes"/>
-<pinref part="RTC1" gate="A" pin="4"/>
+<pinref part="SERIAL" gate="A" pin="4"/>
 </segment>
 </net>
@@
 <wire x1="51.816" y1="87.376" x2="51.816" y2="92.456" width="0.1524" layer="91"/>
 <pinref part="P+6" gate="VCC" pin="VCC"/>
-<pinref part="J1" gate="G$1" pin="2"/>
+<pinref part="ISP" gate="G$1" pin="2"/>
 <junction x="48.514" y="87.376"/>
 </segment>
@@
 <pinref part="P+5" gate="VCC" pin="VCC"/>
 <wire x1="79.756" y1="81.28" x2="97.536" y2="81.28" width="0.1524" layer="91"/>
-<pinref part="RTC1" gate="A" pin="3"/>
+<pinref part="SERIAL" gate="A" pin="3"/>
 </segment>
 <segment>
@@
 <wire x1="51.816" y1="82.296" x2="51.816" y2="77.216" width="0.1524" layer="91"/>
 <pinref part="GND7" gate="1" pin="GND"/>
-<pinref part="J1" gate="G$1" pin="6"/>
+<pinref part="ISP" gate="G$1" pin="6"/>
 <junction x="48.514" y="82.296"/>
 </segment>
@@
 <wire x1="79.756" y1="76.2" x2="89.916" y2="76.2" width="0.1524" layer="91"/>
 <wire x1="89.916" y1="76.2" x2="89.916" y2="71.12" width="0.1524" layer="91"/>
-<pinref part="RTC1" gate="A" pin="1"/>
+<pinref part="SERIAL" gate="A" pin="1"/>
 </segment>
 <segment>
@@
 <wire x1="79.756" y1="88.9" x2="92.456" y2="88.9" width="0.1524" layer="91"/>
 <pinref part="C1" gate="G$1" pin="2"/>
-<pinref part="RTC1" gate="A" pin="6"/>
-</segment>
-</net>
+<pinref part="SERIAL" gate="A" pin="6"/>
+</segment>
+</net>
