File: eagle/keepuntil-v2.0/KeepUntil-v2.0.brd (EAGLE design)
At the start: 37 x 45 mm, 15 parts, among them IC2 REG1117, J2 USBSMD, Q1 CSTCR6M00G53Z, U1 ATMEGA328P-AU

Commit message: working pg app, start v2 board
Parts:
- removed Q1: CSTCR6M00G53Z, murata-filter:CSTCR6M
- added Y1: 8MHZ, SparkFun-FreqCtrl:RESONATOR-SMD
Connections:
- removed net N$1: Q1.1, U1.7
- removed net N$2: Q1.3, U1.8
- net GND: no longer Q1.2
Changed lines of the file:
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@@
 <attribute name="VALUE" x="12.05" y="15.69" size="1.27" layer="27" rot="R90"/>
-</element>
-<element name="Q1" library="murata-filter" package="CSTCR6M" value="CSTCR6M00G53Z" x="11.94" y="24.56" smashed="yes" rot="R270">
-<attribute name="MF" value="" x="11.94" y="24.56" size="1.778" layer="27" rot="R270" display="off"/>
-<attribute name="OC_FARNELL" value="1170434" x="11.94" y="24.56" size="1.778" layer="27" rot="R270" display="off"/>
-<attribute name="OC_NEWARK" value="25M8759" x="11.94" y="24.56" size="1.778" layer="27" rot="R270" display="off"/>
-<attribute name="MPN" value="CSTCR6M00G53-R0" x="11.94" y="24.56" size="1.778" layer="27" rot="R270" display="off"/>
 </element>
 <element name="R1" library="resistor" package="R0805" value="10K" x="9.51" y="11.89" smashed="yes" rot="R90">
@@
 <attribute name="VALUE" x="23.055" y="34.37" size="1.27" layer="27" rot="R270"/>
 </element>
+<element name="Y1" library="SparkFun-FreqCtrl" package="RESONATOR-SMD" value="8MHZ" x="2" y="-3">
+<attribute name="PROD_ID" value="XTAL-08895" x="2" y="-3" size="1.778" layer="27" display="off"/>
+</element>
 </elements>
 <signals>
-<signal name="N$1">
-<contactref element="U1" pad="7"/>
-<contactref element="Q1" pad="1"/>
-<wire x1="11.94" y1="26.06" x2="14.6282" y2="23.8834" width="0" layer="19" extent="1-1"/>
-</signal>
-<signal name="N$2">
-<contactref element="U1" pad="8"/>
-<contactref element="Q1" pad="3"/>
-<wire x1="11.94" y1="23.06" x2="14.6282" y2="23.096" width="0" layer="19" extent="1-1"/>
-</signal>
 <signal name="RESET">
 <contactref element="U1" pad="29"/>
@@
 <contactref element="U1" pad="21"/>
 <contactref element="S1" pad="1"/>
-<contactref element="Q1" pad="2"/>
 <contactref element="J2" pad="GND"/>
 <contactref element="RTC" pad="1"/>
@@
 </polygon>
 <contactref element="JP1" pad="2"/>
-<wire x1="23.1118" y1="26.2964" x2="34.42" y2="37.61" width="0" layer="19" extent="1-1"/>
+<wire x1="28.77" y1="33.1" x2="34.42" y2="37.61" width="0" layer="19" extent="1-1"/>
+<wire x1="23.1118" y1="26.2964" x2="28.77" y2="33.1" width="0" layer="19" extent="1-1"/>
 <wire x1="14.6282" y1="27.0838" x2="23.1118" y2="26.2964" width="0" layer="19" extent="1-1"/>
 <wire x1="14.6282" y1="25.4836" x2="14.6282" y2="27.0838" width="0" layer="19" extent="1-1"/>
-<wire x1="11.94" y1="24.56" x2="14.6282" y2="25.4836" width="0" layer="19" extent="1-1"/>
-<wire x1="6.75" y1="20.65" x2="11.94" y2="24.56" width="0" layer="19" extent="1-1"/>
-<wire x1="9.51" y1="18.382" x2="6.75" y2="20.65" width="0" layer="19" extent="1-1"/>
+<wire x1="9.51" y1="18.382" x2="14.6282" y2="25.4836" width="0" layer="19" extent="1-1"/>
+<wire x1="6.75" y1="20.65" x2="9.51" y2="18.382" width="0" layer="19" extent="1-1"/>
 <wire x1="12.44" y1="12.84" x2="9.51" y2="18.382" width="0" layer="19" extent="1-1"/>
 <wire x1="21.1306" y1="17.5496" x2="23.1118" y2="26.2964" width="0" layer="19" extent="1-1"/>
@@
 <wire x1="20.47" y1="7.43" x2="23.69" y2="13.29" width="0" layer="19" extent="1-1"/>
 <wire x1="9.51" y1="1.89" x2="12.44" y2="12.84" width="0" layer="19" extent="1-1"/>
-<wire x1="28.77" y1="33.1" x2="9.51" y2="1.89" width="0" layer="19" extent="1-1"/>
 <wire x1="8.02" y1="37.61" x2="14.6282" y2="27.0838" width="0" layer="19" extent="1-1"/>
 </signal>
