File: eagle/keepuntil-v2.0/KeepUntil-v2.0.sch (EAGLE design)
At the start: 15 parts, among them IC2 REG1117, J2 USBSMD, Q1 CSTCR6M00G53Z, U1 ATMEGA328P-AU

Commit message: working pg app, start v2 board
Parts:
- removed Q1: CSTCR6M00G53Z, murata-filter:CSTCR6M00G53Z
- added Y1: 8MHZ, SparkFun-FreqCtrl:RESONATOR8MHZ
Connections:
- removed net N$1: Q1.1, U1.PB6
- removed net N$2: Q1.3, U1.PB7
- net GND: no longer Q1.2
Changed lines of the file:
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@@
 </classes>
 <parts>
-<part name="Q1" library="murata-filter" deviceset="CSTCR" device="" technology="6M00G53Z"/>
 <part name="U1" library="Ava" deviceset="ATMEGA328P-AU" device=""/>
 <part name="R1" library="resistor" deviceset="R-EU_" device="R0805" value="10K"/>
@@
 <part name="SERIAL" library="adafruit" deviceset="PINHD-1X6" device="CLEAN"/>
 <part name="JP1" library="pinhead" deviceset="PINHD-2X6" device=""/>
+<part name="Y1" library="SparkFun-FreqCtrl" deviceset="RESONATOR" device="8MHZ" value="8MHZ"/>
 </parts>
 <sheets>
@@
 </plain>
 <instances>
-<instance part="Q1" gate="G$1" x="147.32" y="78.74" smashed="yes" rot="R270">
-<attribute name="NAME" x="151.13" y="83.82" size="1.778" layer="95" rot="R270"/>
-<attribute name="VALUE" x="139.7" y="68.58" size="1.778" layer="96"/>
-</instance>
 <instance part="U1" gate="A" x="190.5" y="96.52"/>
 <instance part="R1" gate="G$1" x="238.76" y="119.38" rot="R90"/>
@@
 <instance part="SERIAL" gate="A" x="77.216" y="83.82" rot="R180"/>
 <instance part="JP1" gate="A" x="73.66" y="48.26"/>
+<instance part="Y1" gate="G$1" x="149.86" y="78.74" rot="R270"/>
 </instances>
 <busses>
 </busses>
 <nets>
-<net name="N$1" class="0">
-<segment>
-<pinref part="U1" gate="A" pin="PB6"/>
-<wire x1="172.72" y1="81.28" x2="157.48" y2="81.28" width="0.1524" layer="91"/>
-<wire x1="157.48" y1="81.28" x2="157.48" y2="86.36" width="0.1524" layer="91"/>
-<pinref part="Q1" gate="G$1" pin="1"/>
-<wire x1="157.48" y1="86.36" x2="147.32" y2="86.36" width="0.1524" layer="91"/>
-</segment>
-</net>
-<net name="N$2" class="0">
-<segment>
-<pinref part="U1" gate="A" pin="PB7"/>
-<wire x1="172.72" y1="78.74" x2="157.48" y2="78.74" width="0.1524" layer="91"/>
-<wire x1="157.48" y1="78.74" x2="157.48" y2="71.12" width="0.1524" layer="91"/>
-<pinref part="Q1" gate="G$1" pin="3"/>
-<wire x1="157.48" y1="71.12" x2="147.32" y2="71.12" width="0.1524" layer="91"/>
-</segment>
-</net>
 <net name="RESET" class="0">
 <segment>
@@
 </segment>
 <segment>
-<pinref part="Q1" gate="G$1" pin="2"/>
-<wire x1="139.7" y1="78.74" x2="134.62" y2="78.74" width="0.1524" layer="91"/>
-<wire x1="134.62" y1="78.74" x2="134.62" y2="66.04" width="0.1524" layer="91"/>
-<pinref part="GND3" gate="1" pin="GND"/>
-</segment>
-<segment>
